Commit message: field work skp

File: urdf/sensors_frogn.xacro (robot description, xacro)
@@ -15,5 +15,5 @@
     <parent link="$(arg tf_prefix)/base_link"/>
     <child link="$(arg tf_prefix)/gps"/>
-    <origin xyz="0.425 -0.875 1.05"/>
+    <origin xyz="0.425 -0.62 1.05"/>
   </joint>
   <!--IMU-->
@@ -58,5 +58,5 @@
       <parent link="$(arg tf_prefix)/base_link"/>
       <child link="$(arg tf_prefix)/camera_bottom_screw_frame" />
-      <origin xyz="-0.425 0.0 1.50" rpy="0 0.366519 0" />
+      <origin xyz="0.735 -0.2 1.205" rpy="0 0.366519 0" />
     </joint>
     <link name="$(arg tf_prefix)/camera_link">
